Commit message: wip

File: urdf/skid_steer_robot.xacro (robot description, xacro)
@@ -1,151 +1,140 @@
 <?xml version="1.0"?>
 <robot xmlns:xacro="http://www.ros.org/wiki/xacro" name="skid_steer_robot">
-  <!-- Include ouster lidar macros -->
-  <xacro:include filename="$(find ouster_gazebo)/urdf/ouster_common.xacro"/>
-  <xacro:include filename="$(find ouster_gazebo)/urdf/ouster_puck.urdf.xacro"/>
-  <!-- Optional chassis and wheel meshes -->
+  <xacro:property name="base_width" value="0.8"/>
+  <xacro:property name="base_length" value="1.2"/>
+  <xacro:property name="base_height" value="0.3"/>
+  <xacro:property name="wheel_radius" value="0.15"/>
+  <xacro:property name="wheel_width" value="0.1"/>
+  <xacro:property name="wheel_offset_x" value="0.4"/>
+  <xacro:property name="wheel_offset_y" value="0.45"/>
+  <xacro:property name="wheel_offset_z" value="-0.05"/>
+  <!-- Base Link -->
   <link name="base_link">
     <visual>
+      <origin xyz="0 0 0" rpy="0 0 0"/>
       <geometry>
-        <box size="0.6 0.4 0.2"/>
+        <box size="${base_length} ${base_width} ${base_height}"/>
       </geometry>
-      <material name="grey"/>
+      <material name="blue">
+        <color rgba="0.2 0.2 0.8 1"/>
+      </material>
     </visual>
     <collision>
+      <origin xyz="0 0 0" rpy="0 0 0"/>
       <geometry>
-        <box size="0.6 0.4 0.2"/>
+        <box size="${base_length} ${base_width} ${base_height}"/>
       </geometry>
     </collision>
     <inertial>
-      <mass value="10.0"/>
-      <inertia ixx="0.1" ixy="0.0" ixz="0.0" iyy="0.1" iyz="0.0" izz="0.1"/>
+      <mass value="50.0"/>
+      <origin xyz="0 0 0" rpy="0 0 0"/>
+      <inertia ixx="4.17" ixy="0.0" ixz="0.0" iyy="6.67" iyz="0.0" izz="8.33"/>
     </inertial>
   </link>
-  <!-- Four wheels, fixed joints with rotation axis -->
-  <link name="wheel_front_left_link">
+  <!-- Wheel Macro -->
+  <xacro:macro name="wheel" params="prefix x_reflect y_reflect">
+    <link name="${prefix}_wheel">
+      <visual>
+        <origin xyz="0 0 0" rpy="1.5708 0 0"/>
+        <geometry>
+          <cylinder radius="${wheel_radius}" length="${wheel_width}"/>
+        </geometry>
+        <material name="black">
+          <color rgba="0.2 0.2 0.2 1"/>
+        </material>
+      </visual>
+      <collision>
+        <origin xyz="0 0 0" rpy="1.5708 0 0"/>
+        <geometry>
+          <cylinder radius="${wheel_radius}" length="${wheel_width}"/>
+        </geometry>
+      </collision>
+      <inertial>
+        <mass value="5.0"/>
+        <origin xyz="0 0 0" rpy="1.5708 0 0"/>
+        <inertia ixx="0.083" ixy="0.0" ixz="0.0" iyy="0.083" iyz="0.0" izz="0.056"/>
+      </inertial>
+    </link>
+    <joint name="${prefix}_wheel_joint" type="continuous">
+      <parent link="base_link"/>
+      <child link="${prefix}_wheel"/>
+      <origin xyz="${x_reflect * wheel_offset_x} ${y_reflect * wheel_offset_y} ${wheel_offset_z}" rpy="0 0 0"/>
+      <axis xyz="0 1 0"/>
+    </joint>
+  </xacro:macro>
+  <!-- Instantiate wheels -->
+  <xacro:wheel prefix="front_left" x_reflect="1" y_reflect="1"/>
+  <xacro:wheel prefix="front_right" x_reflect="1" y_reflect="-1"/>
+  <xacro:wheel prefix="rear_left" x_reflect="-1" y_reflect="1"/>
+  <xacro:wheel prefix="rear_right" x_reflect="-1" y_reflect="-1"/>
+  <!-- Lidar Mount -->
+  <link name="lidar_mount">
     <visual>
+      <origin xyz="0 0 0" rpy="0 0 0"/>
       <geometry>
-        <cylinder length="0.1" radius="0.05"/>
+        <cylinder radius="0.05" length="0.1"/>
       </geometry>
-      <material name="black"/>
+      <material name="gray">
+        <color rgba="0.5 0.5 0.5 1"/>
+      </material>
     </visual>
     <collision>
+      <origin xyz="0 0 0" rpy="0 0 0"/>
       <geometry>
-        <cylinder length="0.1" radius="0.05"/>
+        <cylinder radius="0.05" length="0.1"/>
       </geometry>
     </collision>
     <inertial>
-      <mass value="1.0"/>
-      <inertia ixx="0.01" ixy="0" ixz="0" iyy="0.01" iyz="0" izz="0.01"/>
+      <mass value="0.5"/>
+      <origin xyz="0 0 0" rpy="0 0 0"/>
+      <inertia ixx="0.001" ixy="0.0" ixz="0.0" iyy="0.001" iyz="0.0" izz="0.001"/>
     </inertial>
   </link>
-  <joint name="wheel_front_left_joint" type="continuous">
+  <joint name="lidar_mount_joint" type="fixed">
     <parent link="base_link"/>
-    <child link="wheel_front_left_link"/>
-    <origin xyz="0.25 0.15 0" rpy="0 0 0"/>
-    <axis xyz="0 1 0"/>
+    <child link="lidar_mount"/>
+    <origin xyz="0 0 ${base_height/2 + 0.05}" rpy="0 0 0"/>
   </joint>
-  <link name="wheel_front_right_link">
-    <visual>
-      <geometry>
-        <cylinder length="0.1" radius="0.05"/>
-      </geometry>
-      <material name="black"/>
-    </visual>
-    <collision>
-      <geometry>
-        <cylinder length="0.1" radius="0.05"/>
-      </geometry>
-    </collision>
-    <inertial>
-      <mass value="1.0"/>
-      <inertia ixx="0.01" ixy="0" ixz="0" iyy="0.01" iyz="0" izz="0.01"/>
-    </inertial>
-  </link>
-  <joint name="wheel_front_right_joint" type="continuous">
-    <parent link="base_link"/>
-    <child link="wheel_front_right_link"/>
-    <origin xyz="0.25 -0.15 0" rpy="0 0 0"/>
-    <axis xyz="0 1 0"/>
-  </joint>
-  <link name="wheel_rear_left_link">
-    <visual>
-      <geometry>
-        <cylinder length="0.1" radius="0.05"/>
-      </geometry>
-      <material name="black"/>
-    </visual>
-    <collision>
-      <geometry>
-        <cylinder length="0.1" radius="0.05"/>
-      </geometry>
-    </collision>
-    <inertial>
-      <mass value="1.0"/>
-      <inertia ixx="0.01" ixy="0" ixz="0" iyy="0.01" iyz="0" izz="0.01"/>
-    </inertial>
-  </link>
-  <joint name="wheel_rear_left_joint" type="continuous">
-    <parent link="base_link"/>
-    <child link="wheel_rear_left_link"/>
-    <origin xyz="-0.25 0.15 0" rpy="0 0 0"/>
-    <axis xyz="0 1 0"/>
-  </joint>
-  <link name="wheel_rear_right_link">
-    <visual>
-      <geometry>
-        <cylinder length="0.1" radius="0.05"/>
-      </geometry>
-      <material name="black"/>
-    </visual>
-    <collision>
-      <geometry>
-        <cylinder length="0.1" radius="0.05"/>
-      </geometry>
-    </collision>
-    <inertial>
-      <mass value="1.0"/>
-      <inertia ixx="0.01" ixy="0" ixz="0" iyy="0.01" iyz="0" izz="0.01"/>
-    </inertial>
-  </link>
-  <joint name="wheel_rear_right_joint" type="continuous">
-    <parent link="base_link"/>
-    <child link="wheel_rear_right_link"/>
-    <origin xyz="-0.25 -0.15 0" rpy="0 0 0"/>
-    <axis xyz="0 1 0"/>
-  </joint>
-  <!-- Add the 4 ouster puck lidars using the existing xacro macro -->
-  <xacro:property name="ouster_config" value="$(find ouster_gazebo)/config/ouster_puck.yaml"/>
-  <!-- Front Left Lidar -->
-  <joint name="ouster_puck_fl_joint" type="fixed">
-    <parent link="base_link"/>
-    <child link="ouster_puck_fl_link"/>
-    <origin xyz="0.3 0.2 0.3" rpy="0 0 0"/>
-  </joint>
-  <xacro:ouster_puck name="ouster_puck_fl" config_file="${ouster_config}"/>
-  <!-- Front Right Lidar -->
-  <joint name="ouster_puck_fr_joint" type="fixed">
-    <parent link="base_link"/>
-    <child link="ouster_puck_fr_link"/>
-    <origin xyz="0.3 -0.2 0.3" rpy="0 0 0"/>
-  </joint>
-  <xacro:ouster_puck name="ouster_puck_fr" config_file="${ouster_config}"/>
-  <!-- Rear Left Lidar -->
-  <joint name="ouster_puck_rl_joint" type="fixed">
-    <parent link="base_link"/>
-    <child link="ouster_puck_rl_link"/>
-    <origin xyz="-0.3 0.2 0.3" rpy="0 0 0"/>
-  </joint>
-  <xacro:ouster_puck name="ouster_puck_rl" config_file="${ouster_config}"/>
-  <!-- Rear Right Lidar -->
-  <joint name="ouster_puck_rr_joint" type="fixed">
-    <parent link="base_link"/>
-    <child link="ouster_puck_rr_link"/>
-    <origin xyz="-0.3 -0.2 0.3" rpy="0 0 0"/>
-  </joint>
-  <xacro:ouster_puck name="ouster_puck_rr" config_file="${ouster_config}"/>
-  <!-- Gazebo ros2_control plugin -->
+  <!-- Include Ouster Lidar -->
+  <xacro:include filename="$(find ouster_gazebo)/urdf/ouster_os0.urdf.xacro"/>
+  <xacro:ouster_os0 parent="lidar_mount" name="os0" topic="points">
+    <origin xyz="0 0 0.05" rpy="0 0 0"/>
+  </xacro:ouster_os0>
+  <!-- Gazebo Plugins -->
   <gazebo>
-    <plugin name="ros2_control" filename="libgazebo_ros2_control.so"/>
+    <plugin name="skid_steer_drive_controller" filename="libgazebo_ros_diff_drive.so">
+      <update_rate>100</update_rate>
+      <left_joint>front_left_wheel_joint</left_joint>
+      <left_joint>rear_left_wheel_joint</left_joint>
+      <right_joint>front_right_wheel_joint</right_joint>
+      <right_joint>rear_right_wheel_joint</right_joint>
+      <wheel_separation>0.9</wheel_separation>
+      <wheel_diameter>0.3</wheel_diameter>
+      <max_wheel_torque>100</max_wheel_torque>
+      <max_wheel_acceleration>1.0</max_wheel_acceleration>
+      <command_topic>cmd_vel</command_topic>
+      <odometry_topic>odom</odometry_topic>
+      <odometry_frame>odom</odometry_frame>
+      <robot_base_frame>base_link</robot_base_frame>
+      <publish_odom>true</publish_odom>
+      <publish_odom_tf>true</publish_odom_tf>
+      <publish_wheel_tf>false</publish_wheel_tf>
+    </plugin>
+  </gazebo>
+  <!-- Gazebo colors -->
+  <gazebo reference="base_link">
+    <material>Gazebo/Blue</material>
+  </gazebo>
+  <gazebo reference="front_left_wheel">
+    <material>Gazebo/Black</material>
+  </gazebo>
+  <gazebo reference="front_right_wheel">
+    <material>Gazebo/Black</material>
+  </gazebo>
+  <gazebo reference="rear_left_wheel">
+    <material>Gazebo/Black</material>
+  </gazebo>
+  <gazebo reference="rear_right_wheel">
+    <material>Gazebo/Black</material>
   </gazebo>
 </robot>
